File: keeb-design-files/MCU.sch (KiCad schematic (older format))
At the start: 34 parts, among them J1 Conn_ARM_JTAG_SWD_10, J2 Conn_Coaxial, SW1 SW_Push, U1 STM32L052R8Tx, U2 nRF24L01P, Y1 Crystal, Y2 Crystal

Commit message: Add new Crystal and match symbols and footprints for switches and diodes
Parts:
- removed Y1, Y2: Crystal, symbol Device:Crystal
- added Y1, Y2: Crystal_GND24, Crystal:Crystal_SMD_3225-4Pin_3.2x2.5mm, symbol Device:Crystal_GND24
- SW1: value SW_Push -> RESET
Connections:
- wire segments 162 -> 170
Other:
- moved on the sheet: C20, C21, R3
Changed lines of the file:
@@
 $Descr A4 11693 8268
 encoding utf-8
-Sheet 2 6
+Sheet 2 5
 Title "MCU and RF"
 Date "2020-05-06"
@@
 P 2600 1850
 F 0 "SW1" V 2646 1802 50  0000 R CNN
-F 1 "SW_Push" V 2555 1802 50  0000 R CNN
+F 1 "RESET" V 2555 1802 50  0000 R CNN
 F 2 "Button_Switch_SMD:SW_SPST_B3S-1000" H 2600 2050 50  0001 C CNN
 F 3 "~" H 2600 2050 50  0001 C CNN
@@
 	8900 2600 9000 2600
 Wire Wire Line
-	9000 2600 9000 2800
-Wire Wire Line
 	8900 2400 9300 2400
-Wire Wire Line
-	9300 2400 9300 2800
 $Comp
 L Device:R_Small R3
 U 1 1 5EB83A46
-P 9150 3200
-F 0 "R3" V 8950 3200 50  0000 C CNN
-F 1 "1M" V 9050 3200 50  0000 C CNN
-F 2 "Resistor_SMD:R_0603_1608Metric_Pad1.05x0.95mm_HandSolder" H 9150 3200 50  0001 C CNN
-F 3 "~" H 9150 3200 50  0001 C CNN
-	1    9150 3200
+P 9150 3300
+F 0 "R3" V 9250 3300 50  0000 C CNN
+F 1 "1M" V 9300 3300 50  0000 C CNN
+F 2 "Resistor_SMD:R_0603_1608Metric_Pad1.05x0.95mm_HandSolder" H 9150 3300 50  0001 C CNN
+F 3 "~" H 9150 3300 50  0001 C CNN
+	1    9150 3300
 	0    1    1    0
 $EndComp
 Wire Wire Line
-	9000 2800 9000 3200
-Wire Wire Line
-	9000 3200 9050 3200
-Connection ~ 9000 2800
-Wire Wire Line
-	9000 3200 9000 3350
-Connection ~ 9000 3200
-Wire Wire Line
-	9300 3350 9300 3200
-Connection ~ 9300 2800
-Wire Wire Line
-	9250 3200 9300 3200
-Connection ~ 9300 3200
-Wire Wire Line
-	9300 3200 9300 2800
+	9000 3300 9050 3300
+Wire Wire Line
+	9000 3300 9000 3350
+Connection ~ 9000 3300
+Wire Wire Line
+	9300 3350 9300 3300
+Wire Wire Line
+	9250 3300 9300 3300
+Connection ~ 9300 3300
 $Comp
 L power:GND #PWR0118
@@
 Wire Wire Line
 	600  4750 600  4600
-$Comp
-L Device:Crystal Y2
-U 1 1 5EB7D705
-P 3200 2900
-F 0 "Y2" V 3246 2769 50  0000 R CNN
-F 1 "Crystal" V 3155 2769 50  0000 R CNN
-F 2 "" H 3200 2900 50  0001 C CNN
-F 3 "~" H 3200 2900 50  0001 C CNN
-F 4 "C12668" H 3200 2900 50  0000 C CNN "LCSC Part Number"
-	1    3200 2900
-	0    -1   -1   0
-$EndComp
-Wire Wire Line
-	3200 2750 3700 2750
-Wire Wire Line
-	3700 2750 3700 2850
+Wire Wire Line
+	3700 2700 3700 2850
 Wire Wire Line
 	3700 2850 3750 2850
@@
 	3750 2950 3700 2950
 Wire Wire Line
-	3700 2950 3700 3050
-Wire Wire Line
-	3700 3050 3200 3050
+	3700 2950 3700 3100
 $Comp
 L Device:C_Small C20
 U 1 1 5EB9CC34
-P 2900 2750
-F 0 "C20" V 2671 2750 50  0000 C CNN
-F 1 "14pF" V 2762 2750 50  0000 C CNN
-F 2 "Capacitor_SMD:C_0603_1608Metric_Pad1.05x0.95mm_HandSolder" H 2900 2750 50  0001 C CNN
-F 3 "~" H 2900 2750 50  0001 C CNN
-	1    2900 2750
+P 2900 2700
+F 0 "C20" V 2671 2700 50  0000 C CNN
+F 1 "14pF" V 2762 2700 50  0000 C CNN
+F 2 "Capacitor_SMD:C_0603_1608Metric_Pad1.05x0.95mm_HandSolder" H 2900 2700 50  0001 C CNN
+F 3 "~" H 2900 2700 50  0001 C CNN
+	1    2900 2700
 	0    1    1    0
 $EndComp
-Wire Wire Line
-	3000 2750 3200 2750
-Connection ~ 3200 2750
-Wire Wire Line
-	3000 3050 3200 3050
-Connection ~ 3200 3050
 $Comp
 L power:GND #PWR0126
@@
 	2550 2900 2700 2900
 Wire Wire Line
-	2700 2900 2700 3050
-Wire Wire Line
-	2700 3050 2800 3050
-Wire Wire Line
-	2800 2750 2700 2750
-Wire Wire Line
-	2700 2750 2700 2900
+	2700 2900 2700 3100
+Wire Wire Line
+	2700 3100 2800 3100
+Wire Wire Line
+	2800 2700 2700 2700
+Wire Wire Line
+	2700 2700 2700 2900
 Connection ~ 2700 2900
 $Comp
@@
 $EndComp
 $Comp
-L Device:Crystal Y1
-U 1 1 5EB7CA10
-P 9150 2800
-F 0 "Y1" H 9150 3068 50  0000 C CNN
-F 1 "Crystal" H 9150 2977 50  0000 C CNN
-F 2 "" H 9150 2800 50  0001 C CNN
-F 3 "~" H 9150 2800 50  0001 C CNN
-F 4 "C12668" H 9150 2800 50  0001 C CNN "LCSC Part Number"
-	1    9150 2800
-	1    0    0    -1
-$EndComp
-$Comp
 L Device:C_Small C21
 U 1 1 5EB9DC35
-P 2900 3050
-F 0 "C21" V 2800 3050 50  0000 C CNN
-F 1 "14pF" V 2700 3050 50  0000 C CNN
-F 2 "Capacitor_SMD:C_0603_1608Metric_Pad1.05x0.95mm_HandSolder" H 2900 3050 50  0001 C CNN
-F 3 "~" H 2900 3050 50  0001 C CNN
-	1    2900 3050
+P 2900 3100
+F 0 "C21" V 2800 3100 50  0000 C CNN
+F 1 "14pF" V 2700 3100 50  0000 C CNN
+F 2 "Capacitor_SMD:C_0603_1608Metric_Pad1.05x0.95mm_HandSolder" H 2900 3100 50  0001 C CNN
+F 3 "~" H 2900 3100 50  0001 C CNN
+	1    2900 3100
 	0    -1   -1   0
 $EndComp
+$Comp
+L Device:Crystal_GND24 Y1
+U 1 1 5EBA4261
+P 3250 2900
+F 0 "Y1" V 3100 2700 50  0000 L CNN
+F 1 "Crystal_GND24" V 3250 3144 50  0001 L CNN
+F 2 "Crystal:Crystal_SMD_3225-4Pin_3.2x2.5mm" H 3250 2900 50  0001 C CNN
+F 3 "~" H 3250 2900 50  0001 C CNN
+F 4 "C12668" V 3341 3144 50  0001 L CNN "LCSC Part Number"
+	1    3250 2900
+	0    1    1    0
+$EndComp
+Wire Wire Line
+	3000 3100 3250 3100
+Wire Wire Line
+	3000 2700 3250 2700
+Wire Wire Line
+	3250 2750 3250 2700
+Connection ~ 3250 2700
+Wire Wire Line
+	3250 2700 3700 2700
+Wire Wire Line
+	3250 3050 3250 3100
+Connection ~ 3250 3100
+Wire Wire Line
+	3250 3100 3700 3100
+$Comp
+L power:GND #PWR0127
+U 1 1 5EBE5653
+P 3550 2850
+F 0 "#PWR0127" H 3550 2600 50  0001 C CNN
+F 1 "GND" H 3555 2677 50  0000 C CNN
+F 2 "" H 3550 2850 50  0001 C CNN
+F 3 "" H 3550 2850 50  0001 C CNN
+	1    3550 2850
+	1    0    0    -1
+$EndComp
+Wire Wire Line
+	3550 2850 3450 2850
+Wire Wire Line
+	3450 2850 3450 2900
+Wire Wire Line
+	3050 2900 2700 2900
+Wire Wire Line
+	9000 2600 9000 2700
+Wire Wire Line
+	9300 2400 9300 2700
+$Comp
+L Device:Crystal_GND24 Y2
+U 1 1 5EBF56D8
+P 9150 2700
+F 0 "Y2" H 9344 2791 50  0000 L CNN
+F 1 "Crystal_GND24" H 9344 2700 50  0000 L CNN
+F 2 "Crystal:Crystal_SMD_3225-4Pin_3.2x2.5mm" H 9150 2700 50  0001 C CNN
+F 3 "~" H 9150 2700 50  0001 C CNN
+F 4 "C12668" H 9344 2609 50  0000 L CNN "LCSC Part Number"
+	1    9150 2700
+	1    0    0    -1
+$EndComp
+$Comp
+L power:GND #PWR0128
+U 1 1 5EC142F4
+P 9150 2950
+F 0 "#PWR0128" H 9150 2700 50  0001 C CNN
+F 1 "GND" H 9155 2777 50  0000 C CNN
+F 2 "" H 9150 2950 50  0001 C CNN
+F 3 "" H 9150 2950 50  0001 C CNN
+	1    9150 2950
+	1    0    0    -1
+$EndComp
+Connection ~ 9000 2700
+Connection ~ 9300 2700
+Wire Wire Line
+	9150 2950 9150 2900
+Wire Wire Line
+	9000 2700 9000 3300
+Wire Wire Line
+	9300 2700 9300 3300
+$Comp
+L power:GND #PWR0129
+U 1 1 5EC1D75C
+P 8950 2450
+F 0 "#PWR0129" H 8950 2200 50  0001 C CNN
+F 1 "GND" H 8850 2450 50  0000 C CNN
+F 2 "" H 8950 2450 50  0001 C CNN
+F 3 "" H 8950 2450 50  0001 C CNN
+	1    8950 2450
+	1    0    0    -1
+$EndComp
+Wire Wire Line
+	8950 2450 9150 2450
+Wire Wire Line
+	9150 2450 9150 2500
 $EndSCHEMATC

Commit message: Add ESD diodes, USB isolator and LDO to schematic
Connections:
- net labels added: ROW0, ROW1, ROW2, ROW3, ROW4, USB_D+, USB_D-
- net labels removed: USB_DM, USB_DP
- wire segments 170 -> 175
Changed lines of the file:
@@
 $Descr A4 11693 8268
 encoding utf-8
-Sheet 2 5
+Sheet 5 5
 Title "MCU and RF"
 Date "2020-05-06"
@@
 Connection ~ 4550 1100
 Text HLabel 5150 2750 2    50   Input ~ 0
-USB_DM
+USB_D-
 Text HLabel 5150 2850 2    50   Input ~ 0
-USB_DP
+USB_D+
 Wire Wire Line
 	5150 2750 5050 2750
@@
 Wire Wire Line
 	9150 2450 9150 2500
+Text HLabel 5200 1650 2    50   Input ~ 0
+ROW0
+Text HLabel 5200 1750 2    50   Input ~ 0
+ROW1
+Text HLabel 5200 1850 2    50   Input ~ 0
+ROW2
+Text HLabel 5200 1950 2    50   Input ~ 0
+ROW3
+Text HLabel 5200 2050 2    50   Input ~ 0
+ROW4
+Wire Wire Line
+	5050 1650 5200 1650
+Wire Wire Line
+	5050 1750 5200 1750
+Wire Wire Line
+	5050 1850 5200 1850
+Wire Wire Line
+	5050 1950 5200 1950
+Wire Wire Line
+	5050 2050 5200 2050
 $EndSCHEMATC

Commit message: Start Battery Management and routed matrix to STM32L0
Connections:
- net labels added: COL0, COL1, COL10, COL11, COL12, COL13, COL14, COL2, COL3, COL4, COL5, COL6, COL7, COL8, COL9
- wire segments 175 -> 190
Other:
- note added: "2.4GHz Radio"
- moved on the sheet: C10, C11, C12
Changed lines of the file:
@@
 L Device:C_Small C11
 U 1 1 5EB2E099
-P 6500 1400
-F 0 "C11" H 6592 1446 50  0000 L CNN
-F 1 "0.1uF" H 6592 1355 50  0000 L CNN
-F 2 "Capacitor_SMD:C_0402_1005Metric" H 6500 1400 50  0001 C CNN
-F 3 "~" H 6500 1400 50  0001 C CNN
-F 4 "C1525" H 6500 1400 50  0001 C CNN "LCSC Part Number"
-	1    6500 1400
+P 7750 3700
+F 0 "C11" H 7842 3746 50  0000 L CNN
+F 1 "0.1uF" H 7842 3655 50  0000 L CNN
+F 2 "Capacitor_SMD:C_0402_1005Metric" H 7750 3700 50  0001 C CNN
+F 3 "~" H 7750 3700 50  0001 C CNN
+F 4 "C1525" H 7750 3700 50  0001 C CNN "LCSC Part Number"
+	1    7750 3700
 	1    0    0    -1
 $EndComp
@@
 L Device:C_Small C12
 U 1 1 5EB2E876
-P 6900 1400
-F 0 "C12" H 6992 1446 50  0000 L CNN
-F 1 "1nF" H 6992 1355 50  0000 L CNN
-F 2 "Capacitor_SMD:C_0402_1005Metric" H 6900 1400 50  0001 C CNN
-F 3 "~" H 6900 1400 50  0001 C CNN
-F 4 "C1523" H 6900 1400 50  0001 C CNN "LCSC Part Number"
-	1    6900 1400
+P 8150 3700
+F 0 "C12" H 8242 3746 50  0000 L CNN
+F 1 "1nF" H 8242 3655 50  0000 L CNN
+F 2 "Capacitor_SMD:C_0402_1005Metric" H 8150 3700 50  0001 C CNN
+F 3 "~" H 8150 3700 50  0001 C CNN
+F 4 "C1523" H 8150 3700 50  0001 C CNN "LCSC Part Number"
+	1    8150 3700
 	1    0    0    -1
 $EndComp
@@
 L power:GND #PWR0113
 U 1 1 5EB2F0BC
-P 6700 1600
-F 0 "#PWR0113" H 6700 1350 50  0001 C CNN
-F 1 "GND" H 6705 1427 50  0000 C CNN
-F 2 "" H 6700 1600 50  0001 C CNN
-F 3 "" H 6700 1600 50  0001 C CNN
-	1    6700 1600
-	1    0    0    -1
-$EndComp
-Wire Wire Line
-	6500 1500 6500 1600
-Wire Wire Line
-	6500 1600 6700 1600
-Wire Wire Line
-	6700 1600 6900 1600
-Wire Wire Line
-	6900 1600 6900 1500
-Connection ~ 6700 1600
+P 7950 3900
+F 0 "#PWR0113" H 7950 3650 50  0001 C CNN
+F 1 "GND" H 7955 3727 50  0000 C CNN
+F 2 "" H 7950 3900 50  0001 C CNN
+F 3 "" H 7950 3900 50  0001 C CNN
+	1    7950 3900
+	1    0    0    -1
+$EndComp
+Wire Wire Line
+	7750 3800 7750 3900
+Wire Wire Line
+	7750 3900 7950 3900
+Wire Wire Line
+	7950 3900 8150 3900
+Wire Wire Line
+	8150 3900 8150 3800
+Connection ~ 7950 3900
 $Comp
 L power:+3V3 #PWR0114
 U 1 1 5EB33281
-P 6700 1200
-F 0 "#PWR0114" H 6700 1050 50  0001 C CNN
-F 1 "+3V3" H 6715 1373 50  0000 C CNN
-F 2 "" H 6700 1200 50  0001 C CNN
-F 3 "" H 6700 1200 50  0001 C CNN
-	1    6700 1200
-	1    0    0    -1
-$EndComp
-Wire Wire Line
-	6700 1200 6500 1200
-Wire Wire Line
-	6500 1200 6500 1300
-Wire Wire Line
-	6700 1200 6900 1200
-Wire Wire Line
-	6900 1200 6900 1300
-Connection ~ 6700 1200
+P 7950 3500
+F 0 "#PWR0114" H 7950 3350 50  0001 C CNN
+F 1 "+3V3" H 7965 3673 50  0000 C CNN
+F 2 "" H 7950 3500 50  0001 C CNN
+F 3 "" H 7950 3500 50  0001 C CNN
+	1    7950 3500
+	1    0    0    -1
+$EndComp
+Wire Wire Line
+	7950 3500 7750 3500
+Wire Wire Line
+	7750 3500 7750 3600
+Wire Wire Line
+	7950 3500 8150 3500
+Wire Wire Line
+	8150 3500 8150 3600
+Connection ~ 7950 3500
 $Comp
 L Device:L_Small L1
@@
 L Device:C_Small C10
 U 1 1 5EB9BEBA
-P 6100 1400
-F 0 "C10" H 6192 1446 50  0000 L CNN
-F 1 "4.7uF" H 6192 1355 50  0000 L CNN
-F 2 "Capacitor_SMD:C_0603_1608Metric_Pad1.05x0.95mm_HandSolder" H 6100 1400 50  0001 C CNN
-F 3 "~" H 6100 1400 50  0001 C CNN
-F 4 "C19666" H 6100 1400 50  0001 C CNN "LCSC Part Number"
-	1    6100 1400
-	1    0    0    -1
-$EndComp
-Wire Wire Line
-	6100 1300 6100 1200
-Wire Wire Line
-	6100 1200 6500 1200
-Connection ~ 6500 1200
-Wire Wire Line
-	6100 1500 6100 1600
-Wire Wire Line
-	6100 1600 6500 1600
-Connection ~ 6500 1600
+P 7350 3700
+F 0 "C10" H 7442 3746 50  0000 L CNN
+F 1 "4.7uF" H 7442 3655 50  0000 L CNN
+F 2 "Capacitor_SMD:C_0603_1608Metric_Pad1.05x0.95mm_HandSolder" H 7350 3700 50  0001 C CNN
+F 3 "~" H 7350 3700 50  0001 C CNN
+F 4 "C19666" H 7350 3700 50  0001 C CNN "LCSC Part Number"
+	1    7350 3700
+	1    0    0    -1
+$EndComp
+Wire Wire Line
+	7350 3600 7350 3500
+Wire Wire Line
+	7350 3500 7750 3500
+Connection ~ 7750 3500
+Wire Wire Line
+	7350 3800 7350 3900
+Wire Wire Line
+	7350 3900 7750 3900
+Connection ~ 7750 3900
 Text Label 7550 2200 2    50   ~ 0
 IRQ
@@
 Text Label 7550 2100 2    50   ~ 0
 CE
-Text Label 3650 3350 2    50   ~ 0
+Text Label 5300 2150 2    50   ~ 0
 CE
 Wire Wire Line
-	3650 3350 3750 3350
-Text Label 3650 3450 2    50   ~ 0
+	5300 2150 5050 2150
+Text Label 5300 2250 2    50   ~ 0
 IRQ
 Wire Wire Line
-	3650 3450 3750 3450
+	5300 2250 5050 2250
 $Comp
 L Connector:Conn_ARM_JTAG_SWD_10 J1
@@
 Wire Wire Line
 	9150 2450 9150 2500
-Text HLabel 5200 1650 2    50   Input ~ 0
+Text HLabel 5200 3350 2    50   Input ~ 0
 ROW0
-Text HLabel 5200 1750 2    50   Input ~ 0
+Text HLabel 5200 3450 2    50   Input ~ 0
 ROW1
-Text HLabel 5200 1850 2    50   Input ~ 0
+Text HLabel 5200 3550 2    50   Input ~ 0
 ROW2
-Text HLabel 5200 1950 2    50   Input ~ 0
+Text HLabel 5200 3650 2    50   Input ~ 0
 ROW3
-Text HLabel 5200 2050 2    50   Input ~ 0
+Text HLabel 5200 3750 2    50   Input ~ 0
 ROW4
-Wire Wire Line
-	5050 1650 5200 1650
-Wire Wire Line
-	5050 1750 5200 1750
-Wire Wire Line
-	5050 1850 5200 1850
-Wire Wire Line
-	5050 1950 5200 1950
-Wire Wire Line
-	5050 2050 5200 2050
+Text HLabel 3550 3350 0    50   Output ~ 0
+COL0
+Text HLabel 3550 3450 0    50   Output ~ 0
+COL1
+Text HLabel 3550 3550 0    50   Output ~ 0
+COL2
+Text HLabel 3550 3650 0    50   Output ~ 0
+COL3
+Text HLabel 3550 3750 0    50   Output ~ 0
+COL4
+Text HLabel 3550 3850 0    50   Output ~ 0
+COL5
+Text HLabel 3550 3950 0    50   Output ~ 0
+COL6
+Text HLabel 3550 4050 0    50   Output ~ 0
+COL7
+Text HLabel 3550 4150 0    50   Output ~ 0
+COL8
+Text HLabel 3550 4250 0    50   Output ~ 0
+COL9
+Text HLabel 3550 4350 0    50   Output ~ 0
+COL10
+Text HLabel 3550 4450 0    50   Output ~ 0
+COL11
+Text HLabel 3550 4550 0    50   Output ~ 0
+COL12
+Text HLabel 3550 4650 0    50   Output ~ 0
+COL13
+Text HLabel 3550 4750 0    50   Output ~ 0
+COL14
+Wire Wire Line
+	3550 3350 3750 3350
+Wire Wire Line
+	3750 3450 3550 3450
+Wire Wire Line
+	3750 3550 3550 3550
+Wire Wire Line
+	3750 3650 3550 3650
+Wire Wire Line
+	3750 3750 3550 3750
+Wire Wire Line
+	3750 3850 3550 3850
+Wire Wire Line
+	3750 3950 3550 3950
+Wire Wire Line
+	3750 4050 3550 4050
+Wire Wire Line
+	3750 4150 3550 4150
+Wire Wire Line
+	3750 4250 3550 4250
+Wire Wire Line
+	3750 4350 3550 4350
+Wire Wire Line
+	3750 4450 3550 4450
+Wire Wire Line
+	3750 4550 3550 4550
+Wire Wire Line
+	3750 4650 3550 4650
+Wire Wire Line
+	3750 4750 3550 4750
+Wire Wire Line
+	5200 3350 5050 3350
+Wire Wire Line
+	5050 3450 5200 3450
+Wire Wire Line
+	5050 3550 5200 3550
+Wire Wire Line
+	5050 3650 5200 3650
+Wire Wire Line
+	5050 3750 5200 3750
+Wire Notes Line width 20
+	11100 700  6950 700
+Wire Notes Line width 20
+	6950 700  6950 4300
+Wire Notes Line width 20
+	6950 4300 11050 4300
+Text Notes 10350 4200 0    50   ~ 10
+2.4GHz Radio
 $EndSCHEMATC

Commit message: Add more part #'s, change to STM32L452CEUxx MCU, more layout work
Parts:
- removed C20, C21: 14pF, Capacitor_SMD:C_0603_1608Metric_Pad1.05x0.95mm_HandSolder, symbol Device:C_Small
- removed U1: STM32L052R8Tx, Package_QFP:LQFP-64_10x10mm_P0.5mm, symbol MCU_ST_STM32L0:STM32L052R8Tx
- removed Y1: Crystal_GND24, Crystal:Crystal_SMD_3225-4Pin_3.2x2.5mm, symbol Device:Crystal_GND24
- added R7: 22K, symbol Device:R_Small
- added SW70: BOOT0, Button_Switch_SMD:SW_SPST_B3S-1000, symbol Switch:SW_Push
- added U1: STM32L452CEUx, Package_DFN_QFN:QFN-48-1EP_7x7mm_P0.5mm_EP5.6x5.6mm, symbol MCU_ST_STM32L4:STM32L452CEUx
- C10: footprint Capacitor_SMD:C_0603_1608Metric_Pad1.05x0.95mm_HandSolder -> Capacitor_SMD:C_0603_1608Metric
- C13: footprint Capacitor_SMD:C_0603_1608Metric_Pad1.05x0.95mm_HandSolder -> Capacitor_SMD:C_0402_1005Metric; LCSC Part Number C21117 -> C1585
- C7: footprint Capacitor_SMD:C_0402_1005Metric -> Capacitor_SMD:C_0603_1608Metric; LCSC Part Number C15525 -> C19702
- J2: value Conn_Coaxial -> SMA; footprint Connector_Coaxial:SMA_Amphenol_132289_EdgeMount -> lib_fp:SMA_Amphenol_132289_EdgeMount
- R3: footprint Resistor_SMD:R_0603_1608Metric_Pad1.05x0.95mm_HandSolder -> (none)
Connections:
- net labels added: BOOT0, NRST
- wire segments 190 -> 174
- no-connect marks 2 -> 11
Other:
- moved on the sheet: C9, R1, SW1
