File: keeb-design-files/LEDMatrix.sch (KiCad schematic (older format))
At the start: 24 parts

Commit message: Create gerbers picknplace and bom
Parts:
- C30, C31, C32, C33, C34, C35, C36, C37, C38, C39, C40, C41: LCSC Part Number (none) -> C1525
- D69, D73, D74, D75, D76, D77, D78, D79, D80, D81, D82, D83: LCSC Part Number (none) -> C114586
Changed lines of the file:
@@
 F 2 "LED_SMD:LED_WS2812B_PLCC4_5.0x5.0mm_P3.2mm" H 1550 1200 50  0001 L TNN
 F 3 "https://cdn-shop.adafruit.com/datasheets/WS2812B.pdf" H 1600 1125 50  0001 L TNN
+F 4 "C114586" H 1500 1500 50  0001 C CNN "LCSC Part Number"
 	1    1500 1500
 	1    0    0    -1
@@
 F 2 "LED_SMD:LED_WS2812B_PLCC4_5.0x5.0mm_P3.2mm" H 2550 1200 50  0001 L TNN
 F 3 "https://cdn-shop.adafruit.com/datasheets/WS2812B.pdf" H 2600 1125 50  0001 L TNN
+F 4 "C114586" H 2500 1500 50  0001 C CNN "LCSC Part Number"
 	1    2500 1500
 	1    0    0    -1
@@
 F 2 "LED_SMD:LED_WS2812B_PLCC4_5.0x5.0mm_P3.2mm" H 3550 1200 50  0001 L TNN
 F 3 "https://cdn-shop.adafruit.com/datasheets/WS2812B.pdf" H 3600 1125 50  0001 L TNN
+F 4 "C114586" H 3500 1500 50  0001 C CNN "LCSC Part Number"
 	1    3500 1500
 	1    0    0    -1
@@
 F 2 "LED_SMD:LED_WS2812B_PLCC4_5.0x5.0mm_P3.2mm" H 4550 1200 50  0001 L TNN
 F 3 "https://cdn-shop.adafruit.com/datasheets/WS2812B.pdf" H 4600 1125 50  0001 L TNN
+F 4 "C114586" H 4500 1500 50  0001 C CNN "LCSC Part Number"
 	1    4500 1500
 	1    0    0    -1
@@
 F 2 "LED_SMD:LED_WS2812B_PLCC4_5.0x5.0mm_P3.2mm" H 5550 1200 50  0001 L TNN
 F 3 "https://cdn-shop.adafruit.com/datasheets/WS2812B.pdf" H 5600 1125 50  0001 L TNN
+F 4 "C114586" H 5500 1500 50  0001 C CNN "LCSC Part Number"
 	1    5500 1500
 	1    0    0    -1
@@
 F 2 "LED_SMD:LED_WS2812B_PLCC4_5.0x5.0mm_P3.2mm" H 6550 1200 50  0001 L TNN
 F 3 "https://cdn-shop.adafruit.com/datasheets/WS2812B.pdf" H 6600 1125 50  0001 L TNN
+F 4 "C114586" H 6500 1500 50  0001 C CNN "LCSC Part Number"
 	1    6500 1500
 	1    0    0    -1
@@
 F 2 "LED_SMD:LED_WS2812B_PLCC4_5.0x5.0mm_P3.2mm" H 6550 3050 50  0001 L TNN
 F 3 "https://cdn-shop.adafruit.com/datasheets/WS2812B.pdf" H 6600 2975 50  0001 L TNN
+F 4 "C114586" H 6500 3350 50  0001 C CNN "LCSC Part Number"
 	1    6500 3350
 	-1   0    0    -1
@@
 F 2 "LED_SMD:LED_WS2812B_PLCC4_5.0x5.0mm_P3.2mm" H 5550 3050 50  0001 L TNN
 F 3 "https://cdn-shop.adafruit.com/datasheets/WS2812B.pdf" H 5600 2975 50  0001 L TNN
+F 4 "C114586" H 5500 3350 50  0001 C CNN "LCSC Part Number"
 	1    5500 3350
 	-1   0    0    -1
@@
 F 2 "LED_SMD:LED_WS2812B_PLCC4_5.0x5.0mm_P3.2mm" H 4550 3050 50  0001 L TNN
 F 3 "https://cdn-shop.adafruit.com/datasheets/WS2812B.pdf" H 4600 2975 50  0001 L TNN
+F 4 "C114586" H 4500 3350 50  0001 C CNN "LCSC Part Number"
 	1    4500 3350
 	-1   0    0    -1
@@
 F 2 "LED_SMD:LED_WS2812B_PLCC4_5.0x5.0mm_P3.2mm" H 3550 3050 50  0001 L TNN
 F 3 "https://cdn-shop.adafruit.com/datasheets/WS2812B.pdf" H 3600 2975 50  0001 L TNN
+F 4 "C114586" H 3500 3350 50  0001 C CNN "LCSC Part Number"
 	1    3500 3350
 	-1   0    0    -1
@@
 F 2 "LED_SMD:LED_WS2812B_PLCC4_5.0x5.0mm_P3.2mm" H 2550 3050 50  0001 L TNN
 F 3 "https://cdn-shop.adafruit.com/datasheets/WS2812B.pdf" H 2600 2975 50  0001 L TNN
+F 4 "C114586" H 2500 3350 50  0001 C CNN "LCSC Part Number"
 	1    2500 3350
 	-1   0    0    -1
@@
 F 2 "LED_SMD:LED_WS2812B_PLCC4_5.0x5.0mm_P3.2mm" H 1550 3050 50  0001 L TNN
 F 3 "https://cdn-shop.adafruit.com/datasheets/WS2812B.pdf" H 1600 2975 50  0001 L TNN
+F 4 "C114586" H 1500 3350 50  0001 C CNN "LCSC Part Number"
 	1    1500 3350
 	-1   0    0    -1
@@
 F 2 "Capacitor_SMD:C_0402_1005Metric" H 8000 1400 50  0001 C CNN
 F 3 "~" H 8000 1400 50  0001 C CNN
+F 4 "C1525" H 8000 1400 50  0001 C CNN "LCSC Part Number"
 	1    8000 1400
 	1    0    0    -1
@@
 F 2 "Capacitor_SMD:C_0402_1005Metric" H 8500 1400 50  0001 C CNN
 F 3 "~" H 8500 1400 50  0001 C CNN
+F 4 "C1525" H 8500 1400 50  0001 C CNN "LCSC Part Number"
 	1    8500 1400
 	1    0    0    -1
@@
 F 2 "Capacitor_SMD:C_0402_1005Metric" H 9000 1400 50  0001 C CNN
 F 3 "~" H 9000 1400 50  0001 C CNN
+F 4 "C1525" H 9000 1400 50  0001 C CNN "LCSC Part Number"
 	1    9000 1400
 	1    0    0    -1
@@
 F 2 "Capacitor_SMD:C_0402_1005Metric" H 9500 1400 50  0001 C CNN
 F 3 "~" H 9500 1400 50  0001 C CNN
+F 4 "C1525" H 9500 1400 50  0001 C CNN "LCSC Part Number"
 	1    9500 1400
 	1    0    0    -1
@@
 F 2 "Capacitor_SMD:C_0402_1005Metric" H 10000 1400 50  0001 C CNN
 F 3 "~" H 10000 1400 50  0001 C CNN
+F 4 "C1525" H 10000 1400 50  0001 C CNN "LCSC Part Number"
 	1    10000 1400
 	1    0    0    -1
@@
 F 2 "Capacitor_SMD:C_0402_1005Metric" H 10500 1400 50  0001 C CNN
 F 3 "~" H 10500 1400 50  0001 C CNN
+F 4 "C1525" H 10500 1400 50  0001 C CNN "LCSC Part Number"
 	1    10500 1400
 	1    0    0    -1
@@
 F 2 "Capacitor_SMD:C_0402_1005Metric" H 8000 2550 50  0001 C CNN
 F 3 "~" H 8000 2550 50  0001 C CNN
+F 4 "C1525" H 8000 2550 50  0001 C CNN "LCSC Part Number"
 	1    8000 2550
 	1    0    0    -1
@@
 F 2 "Capacitor_SMD:C_0402_1005Metric" H 8500 2550 50  0001 C CNN
 F 3 "~" H 8500 2550 50  0001 C CNN
+F 4 "C1525" H 8500 2550 50  0001 C CNN "LCSC Part Number"
 	1    8500 2550
 	1    0    0    -1
@@
 F 2 "Capacitor_SMD:C_0402_1005Metric" H 9000 2550 50  0001 C CNN
 F 3 "~" H 9000 2550 50  0001 C CNN
+F 4 "C1525" H 9000 2550 50  0001 C CNN "LCSC Part Number"
 	1    9000 2550
 	1    0    0    -1
@@
 F 2 "Capacitor_SMD:C_0402_1005Metric" H 9500 2550 50  0001 C CNN
 F 3 "~" H 9500 2550 50  0001 C CNN
+F 4 "C1525" H 9500 2550 50  0001 C CNN "LCSC Part Number"
 	1    9500 2550
 	1    0    0    -1
@@
 F 2 "Capacitor_SMD:C_0402_1005Metric" H 10000 2550 50  0001 C CNN
 F 3 "~" H 10000 2550 50  0001 C CNN
+F 4 "C1525" H 10000 2550 50  0001 C CNN "LCSC Part Number"
 	1    10000 2550
 	1    0    0    -1
@@
 F 2 "Capacitor_SMD:C_0402_1005Metric" H 10500 2550 50  0001 C CNN
 F 3 "~" H 10500 2550 50  0001 C CNN
+F 4 "C1525" H 10500 2550 50  0001 C CNN "LCSC Part Number"
 	1    10500 2550
 	1    0    0    -1

Commit message: Re-Generate Gerbers
Parts:
- D69, D73, D74, D75, D76, D77, D78, D79, D80, D81, D82, D83: footprint LED_SMD:LED_WS2812B_PLCC4_5.0x5.0mm_P3.2mm -> lib_fp:LED_WS2812B_PLCC4_5.0x5.0mm_P3.2mm
Changed lines of the file:
@@
 F 0 "D69" H 1844 1546 50  0000 L CNN
 F 1 "WS2812B" H 1844 1455 50  0000 L CNN
-F 2 "LED_SMD:LED_WS2812B_PLCC4_5.0x5.0mm_P3.2mm" H 1550 1200 50  0001 L TNN
+F 2 "lib_fp:LED_WS2812B_PLCC4_5.0x5.0mm_P3.2mm" H 1550 1200 50  0001 L TNN
 F 3 "https://cdn-shop.adafruit.com/datasheets/WS2812B.pdf" H 1600 1125 50  0001 L TNN
 F 4 "C114586" H 1500 1500 50  0001 C CNN "LCSC Part Number"
@@
 F 0 "D74" H 2844 1546 50  0000 L CNN
 F 1 "WS2812B" H 2844 1455 50  0000 L CNN
-F 2 "LED_SMD:LED_WS2812B_PLCC4_5.0x5.0mm_P3.2mm" H 2550 1200 50  0001 L TNN
+F 2 "lib_fp:LED_WS2812B_PLCC4_5.0x5.0mm_P3.2mm" H 2550 1200 50  0001 L TNN
 F 3 "https://cdn-shop.adafruit.com/datasheets/WS2812B.pdf" H 2600 1125 50  0001 L TNN
 F 4 "C114586" H 2500 1500 50  0001 C CNN "LCSC Part Number"
@@
 F 0 "D76" H 3844 1546 50  0000 L CNN
 F 1 "WS2812B" H 3844 1455 50  0000 L CNN
-F 2 "LED_SMD:LED_WS2812B_PLCC4_5.0x5.0mm_P3.2mm" H 3550 1200 50  0001 L TNN
+F 2 "lib_fp:LED_WS2812B_PLCC4_5.0x5.0mm_P3.2mm" H 3550 1200 50  0001 L TNN
 F 3 "https://cdn-shop.adafruit.com/datasheets/WS2812B.pdf" H 3600 1125 50  0001 L TNN
 F 4 "C114586" H 3500 1500 50  0001 C CNN "LCSC Part Number"
@@
 F 0 "D78" H 4844 1546 50  0000 L CNN
 F 1 "WS2812B" H 4844 1455 50  0000 L CNN
-F 2 "LED_SMD:LED_WS2812B_PLCC4_5.0x5.0mm_P3.2mm" H 4550 1200 50  0001 L TNN
+F 2 "lib_fp:LED_WS2812B_PLCC4_5.0x5.0mm_P3.2mm" H 4550 1200 50  0001 L TNN
 F 3 "https://cdn-shop.adafruit.com/datasheets/WS2812B.pdf" H 4600 1125 50  0001 L TNN
 F 4 "C114586" H 4500 1500 50  0001 C CNN "LCSC Part Number"
@@
 F 0 "D81" H 5844 1546 50  0000 L CNN
 F 1 "WS2812B" H 5844 1455 50  0000 L CNN
-F 2 "LED_SMD:LED_WS2812B_PLCC4_5.0x5.0mm_P3.2mm" H 5550 1200 50  0001 L TNN
+F 2 "lib_fp:LED_WS2812B_PLCC4_5.0x5.0mm_P3.2mm" H 5550 1200 50  0001 L TNN
 F 3 "https://cdn-shop.adafruit.com/datasheets/WS2812B.pdf" H 5600 1125 50  0001 L TNN
 F 4 "C114586" H 5500 1500 50  0001 C CNN "LCSC Part Number"
@@
 F 0 "D82" H 6844 1546 50  0000 L CNN
 F 1 "WS2812B" H 6844 1455 50  0000 L CNN
-F 2 "LED_SMD:LED_WS2812B_PLCC4_5.0x5.0mm_P3.2mm" H 6550 1200 50  0001 L TNN
+F 2 "lib_fp:LED_WS2812B_PLCC4_5.0x5.0mm_P3.2mm" H 6550 1200 50  0001 L TNN
 F 3 "https://cdn-shop.adafruit.com/datasheets/WS2812B.pdf" H 6600 1125 50  0001 L TNN
 F 4 "C114586" H 6500 1500 50  0001 C CNN "LCSC Part Number"
@@
 F 0 "D83" H 6844 3396 50  0000 L CNN
 F 1 "WS2812B" H 6844 3305 50  0000 L CNN
-F 2 "LED_SMD:LED_WS2812B_PLCC4_5.0x5.0mm_P3.2mm" H 6550 3050 50  0001 L TNN
+F 2 "lib_fp:LED_WS2812B_PLCC4_5.0x5.0mm_P3.2mm" H 6550 3050 50  0001 L TNN
 F 3 "https://cdn-shop.adafruit.com/datasheets/WS2812B.pdf" H 6600 2975 50  0001 L TNN
 F 4 "C114586" H 6500 3350 50  0001 C CNN "LCSC Part Number"
@@
 F 0 "D80" H 5844 3396 50  0000 L CNN
 F 1 "WS2812B" H 5844 3305 50  0000 L CNN
-F 2 "LED_SMD:LED_WS2812B_PLCC4_5.0x5.0mm_P3.2mm" H 5550 3050 50  0001 L TNN
+F 2 "lib_fp:LED_WS2812B_PLCC4_5.0x5.0mm_P3.2mm" H 5550 3050 50  0001 L TNN
 F 3 "https://cdn-shop.adafruit.com/datasheets/WS2812B.pdf" H 5600 2975 50  0001 L TNN
 F 4 "C114586" H 5500 3350 50  0001 C CNN "LCSC Part Number"
@@
 F 0 "D79" H 4844 3396 50  0000 L CNN
 F 1 "WS2812B" H 4844 3305 50  0000 L CNN
-F 2 "LED_SMD:LED_WS2812B_PLCC4_5.0x5.0mm_P3.2mm" H 4550 3050 50  0001 L TNN
+F 2 "lib_fp:LED_WS2812B_PLCC4_5.0x5.0mm_P3.2mm" H 4550 3050 50  0001 L TNN
 F 3 "https://cdn-shop.adafruit.com/datasheets/WS2812B.pdf" H 4600 2975 50  0001 L TNN
 F 4 "C114586" H 4500 3350 50  0001 C CNN "LCSC Part Number"
@@
 F 0 "D77" H 3844 3396 50  0000 L CNN
 F 1 "WS2812B" H 3844 3305 50  0000 L CNN
-F 2 "LED_SMD:LED_WS2812B_PLCC4_5.0x5.0mm_P3.2mm" H 3550 3050 50  0001 L TNN
+F 2 "lib_fp:LED_WS2812B_PLCC4_5.0x5.0mm_P3.2mm" H 3550 3050 50  0001 L TNN
 F 3 "https://cdn-shop.adafruit.com/datasheets/WS2812B.pdf" H 3600 2975 50  0001 L TNN
 F 4 "C114586" H 3500 3350 50  0001 C CNN "LCSC Part Number"
@@
 F 0 "D75" H 2844 3396 50  0000 L CNN
 F 1 "WS2812B" H 2844 3305 50  0000 L CNN
-F 2 "LED_SMD:LED_WS2812B_PLCC4_5.0x5.0mm_P3.2mm" H 2550 3050 50  0001 L TNN
+F 2 "lib_fp:LED_WS2812B_PLCC4_5.0x5.0mm_P3.2mm" H 2550 3050 50  0001 L TNN
 F 3 "https://cdn-shop.adafruit.com/datasheets/WS2812B.pdf" H 2600 2975 50  0001 L TNN
 F 4 "C114586" H 2500 3350 50  0001 C CNN "LCSC Part Number"
@@
 F 0 "D73" H 1844 3396 50  0000 L CNN
 F 1 "WS2812B" H 1844 3305 50  0000 L CNN
-F 2 "LED_SMD:LED_WS2812B_PLCC4_5.0x5.0mm_P3.2mm" H 1550 3050 50  0001 L TNN
+F 2 "lib_fp:LED_WS2812B_PLCC4_5.0x5.0mm_P3.2mm" H 1550 3050 50  0001 L TNN
 F 3 "https://cdn-shop.adafruit.com/datasheets/WS2812B.pdf" H 1600 2975 50  0001 L TNN
 F 4 "C114586" H 1500 3350 50  0001 C CNN "LCSC Part Number"
