File: keeb-design-files/keeb.kicad_pcb (KiCad board)
At the start: 2 copper layers, 307.3 x 115.6 mm, 183 parts, among them J1 Conn_ARM_JTAG_SWD_10, J2 SMA, J3 USB_B, Q1 DMG3415U, SW1 RESET, SW10 8, SW11 9, SW12 0, SW13 -, SW14 =, SW15 BACKSPACE, SW16 HOME, SW17 TAB, SW18 CAPS LOCK, SW19 L_SHIFT, SW2 `, SW20 L_CTRL, SW21 Q, SW22 A, SW23 Z, SW24 WIN, SW25 W, SW26 S, SW27 X, SW28 L_ALT, SW29 E, SW3 1, SW30 D, SW31 C, SW32 SPACE, SW33 R, SW34 F, SW35 V, SW36 R_ALT, SW37 T, SW38 G, SW39 B, SW4 2, SW40 FN, SW41 Y, SW42 H, SW43 N, SW44 R_CTRL, SW45 U, SW46 J, SW47 M, SW48 LEFT, SW49 I, SW5 3, SW50 K, SW51 ,, SW52 DOWN, SW53 O, SW54 L, SW55 ., SW56 RIGHT, SW57 P, SW58 ;, SW59 /, SW6 4, SW60 [, SW61 ', SW62 R_SHIFT, SW63 ], SW64 ENTER, SW65 UP, SW66 \, SW67 PAGE DOWN, SW68 END, SW69 PAGE UP, SW7 5, SW70 BOOT0, SW8 6, SW9 7, U1 STM32L452CEUx, U2 nRF24L01P, U3 USBLC6-2SC6, U4 BQ24075, U5 NXE2S0505MC, Y2 Crystal_GND24

Commit message: Connect USB Hierarchical pins to MCU
Parts:
- moved D2 2.65 mm to (54.9, 80.0)
- moved D64 0.98 mm to (312.2, 80.0)
- moved D7 0.97 mm to (78.7, 80.0)
- moved D12 0.96 mm to (97.5, 80.0)
- moved D68 0.95 mm to (335.8, 80.0)
- moved D17 0.95 mm to (116.7, 80.0)
- moved D22 0.95 mm to (135.7, 80.0)
- moved D27 0.95 mm to (154.8, 80.0)
- moved D32 0.95 mm to (173.8, 80.0)
- moved D37 0.95 mm to (192.9, 80.0)
- moved D42 0.95 mm to (211.9, 80.0)
- moved D47 0.95 mm to (231.0, 80.0)
- moved D52 0.95 mm to (250.0, 80.0)
- moved D56 0.95 mm to (269.1, 80.0)
- moved D60 0.95 mm to (288.1, 80.0)
Routing:
- net /MCU/ROW2: track 0.00 -> 280.4 mm
- net /MCU/ROW3: track 0.00 -> 274.6 mm
- net Net-(D2-Pad2): track 7.58 -> 4.92 mm
- net /MCU/ROW1: track 283.4 -> 282.0 mm
- net Net-(D22-Pad2): track 6.08 -> 5.08 mm
- net Net-(D37-Pad2): track 6.08 -> 5.10 mm
- net Net-(D27-Pad2): track 6.08 -> 5.10 mm
- net Net-(D17-Pad2): track 6.08 -> 5.12 mm
- net Net-(D52-Pad2): track 6.08 -> 5.12 mm
- net Net-(D32-Pad2): track 6.08 -> 5.14 mm
- net Net-(D47-Pad2): track 6.08 -> 5.14 mm
- net Net-(D42-Pad2): track 6.08 -> 5.14 mm
- net Net-(D7-Pad2): track 6.08 -> 5.15 mm
- net Net-(D64-Pad2): track 6.08 -> 5.15 mm
- net Net-(D60-Pad2): track 6.08 -> 5.18 mm
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
Commit message: Confirm LCSC part numbers, started placement for layout
Parts:
- removed Q1: DMG3415U, Package_TO_SOT_SMD:SOT-23
- added C20: 0.1uF, Capacitor_SMD:C_0402_1005Metric, B.Cu at (86.1, 68.6)
- added C21: 1uF, Capacitor_SMD:C_0402_1005Metric, B.Cu at (87.1, 66.5)
- added C22: 1uF, Capacitor_SMD:C_0402_1005Metric, B.Cu at (100.8, 66.8)
- added C27: 1uF, Capacitor_SMD:C_0402_1005Metric, B.Cu at (86.6, 72.4)
- added C28: 1uF, Capacitor_SMD:C_0402_1005Metric, B.Cu at (80.5, 74.4)
- added C29: 0.1uF, Capacitor_SMD:C_0402_1005Metric, B.Cu at (84.8, 68.6)
- added D72: G_LED, LED_SMD:LED_0603_1608Metric, F.Cu at (107.4, 71.9)
- added FB1: 100 @ 100MHz, Resistor_SMD:R_0603_1608Metric_Pad1.05x0.95mm_HandSolder, B.Cu at (66.5, 52.2)
- added J4: S2B-PH-K-S, Connector_JST:JST_PH_S2B-PH-K_1x02_P2.00mm_Horizontal, B.Cu at (104.4, 10.9)
- added J5: Conn_01x02, Connector_JST:JST_PH_S2B-PH-K_1x02_P2.00mm_Horizontal, F.Cu at (283.4, -25.5)
- added J6: Conn_01x04, lib_fp:OLED_Display, F.Cu at (103.9, 43.9)
- added L4: 15uH, Inductor_SMD:L_Bourns_SRR1260, B.Cu at (88.1, 55.9)
- added L5: 22uH, Inductor_SMD:L_Bourns_SRR1260, B.Cu at (116.1, 55.6)
- added R10: 10K, Resistor_SMD:R_0603_1608Metric_Pad1.05x0.95mm_HandSolder, F.Cu at (298.3, -31.0)
- added R11: 100R, Resistor_SMD:R_0402_1005Metric, B.Cu at (105.4, 69.1)
- added R12: 100R, Resistor_SMD:R_0402_1005Metric, B.Cu at (107.4, 69.1)
- added R13: 100K, Resistor_SMD:R_0402_1005Metric, B.Cu at (80.8, 66.3)
- added R14: 30m, Resistor_SMD:R_0805_2012Metric, B.Cu at (89.4, 65.5)
- added R15: 1.1K, Resistor_SMD:R_0402_1005Metric, B.Cu at (85.9, 66.5)
- added R16: 3.3K, Resistor_SMD:R_0603_1608Metric_Pad1.05x0.95mm_HandSolder, B.Cu at (77.2, 61.0)
- added R17: 3.3K, Resistor_SMD:R_0603_1608Metric_Pad1.05x0.95mm_HandSolder, B.Cu at (79.0, 61.0)
- added R18: 100K, Resistor_SMD:R_0402_1005Metric, B.Cu at (79.8, 66.3)
- added R7: 22K, Resistor_SMD:R_0402_1005Metric, F.Cu at (302.2, -73.2)
- added R8: 820R, Resistor_SMD:R_0402_1005Metric, B.Cu at (100.8, 69.6)
- added R9: 100K, Resistor_SMD:R_0402_1005Metric, B.Cu at (119.1, 64.8)
- added SW71: SW_SPDT, lib_fp:SW_CuK_OS102011MA1QN1_SPDT_Angled, F.Cu at (132.1, 44.5)
- added U6: STC3100, Package_DFN_QFN:DFN-8-1EP_3x3mm_P0.5mm_EP1.66x2.38mm, B.Cu at (83.3, 65.5)
- added U7: LD39050P, Package_DFN_QFN:DFN-6-1EP_3x3mm_P0.95mm_EP1.7x2.6mm, B.Cu at (83.6, 73.4)
- C24, C26, R4, R5, U5: moved to B.Cu
- C25: value 4.7uF -> 10uF
- D71: value MBR120 -> Y_LED; footprint Diode_SMD:D_SOD-123F -> LED_SMD:LED_0603_1608Metric
- R6: value 100K -> 1.1K; moved to B.Cu
- U4: footprint Package_DFN_QFN:QFN-16-1EP_3x3mm_P0.5mm_EP1.7x1.7mm -> lib_fp:QFN-16-1EP_3x3mm_P0.5mm_EP1.7x1.7mm; moved to B.Cu
- moved D71 456.9 mm to (105.4, 71.9), turned to 270 degrees
- moved J1 135.5 mm to (30.2, 67.6)
- moved C26 117.5 mm to (119.6, 63.2)
- moved U4 68.1 mm to (98.0, 67.8), turned to 90 degrees
- moved D69 67.7 mm to (82.8, 51.6)
- moved C24 61.4 mm to (90.4, 63.2)
- moved J3 46.0 mm to (70.1, 48.5)
- moved C7 42.2 mm to (62.7, 69.6), turned to 180 degrees
- moved U3 41.9 mm to (71.4, 62.2), turned to 90 degrees
- moved R6 40.3 mm to (99.8, 65.0)
- moved R5 37.3 mm to (123.4, 51.6), turned to 270 degrees
- moved U5 36.5 mm to (102.1, 55.9), turned to 0 degrees
- moved C5 34.7 mm to (75.2, 71.5)
- moved C14 34.6 mm to (47.2, 64.5), turned to 180 degrees
- moved C1 34.6 mm to (65.7, 67.4)
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Connections:
- net /USB and Power Management/BAT_INPUT renamed /USB and Power Management/BAT_IN
- D71 pad 2: +5V -> +BATT
- R6 pad 1: +5V -> Net-(R6-Pad1)
- U1 pad 26: Net-(U1-Pad26) -> /MCU/EN1
- U1 pad 29: Net-(U1-Pad29) -> /MCU/EN2
- U1 pad 30: Net-(U1-Pad30) -> /MCU/SCL_MON
- U1 pad 31: Net-(U1-Pad31) -> /MCU/SDA_MON
- U1 pad 38: Net-(U1-Pad38) -> /MCU/~CE~
- U4 pad 12: Net-(U4-Pad12) -> Net-(R6-Pad1)
- U4 pad 15: +5V -> /USB and Power Management/SYS_OFF
- U4 pad 4: Net-(U4-Pad4) -> /MCU/~CE~
- U4 pad 5: Net-(U4-Pad5) -> /MCU/EN2
- U4 pad 6: Net-(U4-Pad6) -> /MCU/EN1
Routing:
- net GND: vias 0 -> 30
- net (no net): vias 0 -> 4
Other:
- board size 307.3 x 115.6 mm -> 309.1 x 131.1 mm

Commit message: More placement before layout
Parts:
- C23, C25, C3, J5, R10, R3: moved to B.Cu
- moved C6 340.5 mm to (25.1, 53.1)
- moved C9 331.2 mm to (21.3, 78.2)
- moved R1 328.0 mm to (20.8, 83.1)
- moved R7 311.5 mm to (23.9, 66.8)
- moved C3 309.8 mm to (62.5, 67.8), turned to 180 degrees
- moved SW1 300.5 mm to (29.5, 80.3)
- moved R3 297.7 mm to (52.6, 61.5), turned to 270 degrees
- moved SW70 223.8 mm to (31.5, 68.6)
- moved R10 201.8 mm to (121.9, 67.1), turned to 90 degrees
- moved J5 179.6 mm to (128.0, 64.5), turned to 270 degrees
- moved C25 120.8 mm to (98.3, 64.3), turned to 180 degrees
- moved C23 120.2 mm to (99.1, 71.4), turned to 270 degrees
- moved J4 60.5 mm to (104.9, 71.4), turned to 270 degrees
- moved J1 14.2 mm to (30.5, 53.3)
- moved D72 8.13 mm to (115.6, 71.9)
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Connections:
- U6 pad 9: (no net) -> GND
Routing:
- net GND: vias 30 -> 40
Other:
- board size 309.1 x 131.1 mm -> 317.5 x 134.6 mm

Commit message: Re-map MCU pins, Add LEDs, Remove USB Isolation cause it couldn't handle the POWER! More routing done
Parts:
- removed L4: 15uH, Inductor_SMD:L_Bourns_SRR1260
- removed L5: 22uH, Inductor_SMD:L_Bourns_SRR1260
- removed R4: 100R, Resistor_SMD:R_0402_1005Metric
- removed U5: NXE2S0505MC, Converter_DCDC:Converter_DCDC_muRata_NXE2SxxxxMC_THT
- added C30: 0.1uF, Capacitor_SMD:C_0402_1005Metric, B.Cu at (68.8, 148.6)
- added C31: 0.1uF, Capacitor_SMD:C_0402_1005Metric, B.Cu at (79.8, 91.9)
- added C32: 0.1uF, Capacitor_SMD:C_0402_1005Metric, B.Cu at (124.5, 91.9)
- added C33: 0.1uF, Capacitor_SMD:C_0402_1005Metric, B.Cu at (172.0, 149.6)
- added C34: 0.1uF, Capacitor_SMD:C_0402_1005Metric, B.Cu at (180.1, 91.7)
- added C35: 0.1uF, Capacitor_SMD:C_0402_1005Metric, B.Cu at (230.4, 92.2)
- added C36: 0.1uF, Capacitor_SMD:C_0402_1005Metric, B.Cu at (215.4, 149.6)
- added C37: 0.1uF, Capacitor_SMD:C_0402_1005Metric, B.Cu at (114.0, 149.4)
- added C38: 0.1uF, Capacitor_SMD:C_0402_1005Metric, B.Cu at (274.3, 91.7)
- added C39: 0.1uF, Capacitor_SMD:C_0402_1005Metric, B.Cu at (267.5, 149.1)
- added C40: 0.1uF, Capacitor_SMD:C_0402_1005Metric, B.Cu at (317.2, 148.6)
- added C41: 0.1uF, Capacitor_SMD:C_0402_1005Metric, B.Cu at (318.3, 87.6)
- added D73: WS2812B, LED_SMD:LED_WS2812B_PLCC4_5.0x5.0mm_P3.2mm, B.Cu at (73.2, 148.6)
- added D74: WS2812B, LED_SMD:LED_WS2812B_PLCC4_5.0x5.0mm_P3.2mm, B.Cu at (120.1, 91.4)
- added D75: WS2812B, LED_SMD:LED_WS2812B_PLCC4_5.0x5.0mm_P3.2mm, B.Cu at (118.4, 148.6)
- added D76: WS2812B, LED_SMD:LED_WS2812B_PLCC4_5.0x5.0mm_P3.2mm, B.Cu at (175.8, 91.7)
- added D77: WS2812B, LED_SMD:LED_WS2812B_PLCC4_5.0x5.0mm_P3.2mm, B.Cu at (176.3, 148.6)
- added D78: WS2812B, LED_SMD:LED_WS2812B_PLCC4_5.0x5.0mm_P3.2mm, B.Cu at (226.1, 91.9)
- added D79: WS2812B, LED_SMD:LED_WS2812B_PLCC4_5.0x5.0mm_P3.2mm, B.Cu at (219.7, 148.6)
- added D80: WS2812B, LED_SMD:LED_WS2812B_PLCC4_5.0x5.0mm_P3.2mm, B.Cu at (271.8, 148.6)
- added D81: WS2812B, LED_SMD:LED_WS2812B_PLCC4_5.0x5.0mm_P3.2mm, B.Cu at (270.0, 91.7)
- added D82: WS2812B, LED_SMD:LED_WS2812B_PLCC4_5.0x5.0mm_P3.2mm, B.Cu at (318.3, 91.4)
- added D83: WS2812B, LED_SMD:LED_WS2812B_PLCC4_5.0x5.0mm_P3.2mm, B.Cu at (321.6, 148.6)
- C6, C9, R1, R7: moved to B.Cu
- D69: value Y_LED -> WS2812B; footprint LED_SMD:LED_0603_1608Metric -> LED_SMD:LED_WS2812B_PLCC4_5.0x5.0mm_P3.2mm; moved to B.Cu
- FB1: value 100 @ 100MHz -> 60 @ 100MHz
- J4: value S2B-PH-K-S -> S2B-PH-SM4-TB; footprint Connector_JST:JST_PH_S2B-PH-K_1x02_P2.00mm_Horizontal -> lib_fp:JST_PH_S2B-PH-SM4-TB_1x02-1MP_P2.00mm_Horizontal
- J5: value Conn_01x02 -> S2B-PH-SM4-TB; footprint Connector_JST:JST_PH_S2B-PH-K_1x02_P2.00mm_Horizontal -> lib_fp:JST_PH_S2B-PH-SM4-TB_1x02-1MP_P2.00mm_Horizontal
- SW1, SW70: footprint Button_Switch_SMD:SW_SPST_B3S-1000 -> lib_fp:SW_SPST_B3S-1000
- moved C26 55.2 mm to (69.1, 42.9), turned to 270 degrees
- moved R1 50.1 mm to (62.7, 55.6), turned to 270 degrees
- moved R5 49.3 mm to (75.2, 51.1)
- moved C9 46.1 mm to (61.5, 55.6), turned to 90 degrees
- moved C6 46.1 mm to (67.3, 71.6), turned to 180 degrees
- moved D70 46.0 mm to (75.9, 48.3)
- moved J5 45.9 mm to (82.3, 59.9), turned to 90 degrees
- moved J1 45.6 mm to (72.9, 70.1)
- moved D69 42.0 mm to (75.4, 91.9), turned to 180 degrees
- moved SW1 41.8 mm to (63.2, 55.6)
- moved C24 31.2 mm to (67.3, 42.9), turned to 270 degrees
- moved J4 30.7 mm to (82.3, 50.5), turned to 90 degrees
- moved R10 29.7 mm to (93.5, 58.7), turned to 180 degrees
- moved SW71 27.7 mm to (108.5, 56.6), turned to 90 degrees
- moved D72 23.9 mm to (91.7, 70.6)
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Connections:
- C24 pad 1: Net-(C24-Pad1) -> +5V
- C24 pad 2: Earth -> GND
- D69 pad 1: Net-(D69-Pad1) -> +3V3
- D69 pad 2: Net-(C24-Pad1) -> Net-(D69-Pad2)
- FB1 pad 1: Net-(C24-Pad1) -> +5V
- J3 pad 4: Earth -> GND
- SW56 pad 2: /MCU/COL9 -> /MCU/COL14
- SW67 pad 2: /MCU/COL13 -> /MCU/COL14
- SW68 pad 2: /MCU/COL13 -> /MCU/COL14
- U1 pad 10: /MCU/COL0 -> /MCU/~CE~
- U1 pad 11: /MCU/COL1 -> /MCU/SPI_SCK
- U1 pad 12: /MCU/COL2 -> Net-(U1-Pad12)
- U1 pad 13: /MCU/COL3 -> /MCU/IRQ
- U1 pad 14: /MCU/COL4 -> /MCU/SPI_NSS
- U1 pad 15: /MCU/COL5 -> /MCU/CE
- U1 pad 16: /MCU/COL6 -> /MCU/SPI_MISO
- U1 pad 17: /MCU/COL7 -> /MCU/SPI_MOSI
- U1 pad 18: /MCU/ROW0 -> /MCU/COL14
- U1 pad 19: /MCU/ROW1 -> /MCU/COL13
- U1 pad 2: /MCU/COL8 -> /MCU/ROW2
- U1 pad 20: /MCU/ROW2 -> /MCU/COL12
- U1 pad 21: /MCU/SPI_SCK -> /MCU/COL11
- U1 pad 22: /MCU/IRQ -> /MCU/COL10
- U1 pad 25: /MCU/SPI_NSS -> /MCU/COL9
- U1 pad 26: /MCU/EN1 -> /MCU/COL8
- U1 pad 27: /MCU/SPI_MISO -> /MCU/COL7
- U1 pad 28: /MCU/SPI_MOSI -> /MCU/COL6
- U1 pad 29: /MCU/EN2 -> /MCU/COL5
- U1 pad 3: /MCU/COL9 -> /MCU/ROW3
- U1 pad 38: /MCU/~CE~ -> /MCU/COL4
- U1 pad 39: /MCU/ROW3 -> /MCU/COL3
- U1 pad 4: /MCU/COL10 -> /MCU/ROW4
- U1 pad 40: /MCU/ROW4 -> /MCU/COL2
- U1 pad 41: /MCU/COL11 -> /MCU/COL1
- U1 pad 42: /MCU/COL12 -> /MCU/COL0
- U1 pad 43: /MCU/COL13 -> /LED Matrix/LED_DIN
- U1 pad 45: /MCU/COL14 -> /MCU/ROW0
- U1 pad 46: /MCU/CE -> /MCU/ROW1
- U1 pad 5: Net-(U1-Pad5) -> /MCU/EN1
- U1 pad 6: Net-(U1-Pad6) -> /MCU/EN2
- U3 pad 2: Earth -> GND
- U3 pad 5: Net-(C24-Pad1) -> +5V
- U6 pad 9: GND -> (no net)
Routing:
- net /MCU/COL14: track 0.00 -> 392.3 mm, vias 0 -> 2
- net /MCU/COL13: track 0.00 -> 277.4 mm, vias 0 -> 2
- net /MCU/ROW0: track 286.2 -> 30.1 mm
- net /MCU/COL12: track 0.00 -> 248.7 mm, vias 0 -> 2
- net /MCU/ROW1: track 282.0 -> 51.0 mm
- net /MCU/COL11: track 0.00 -> 228.4 mm, vias 0 -> 2
- net /MCU/ROW2: track 280.4 -> 71.1 mm
- net /MCU/COL10: track 0.00 -> 207.0 mm, vias 0 -> 2
- net /MCU/COL9: track 0.00 -> 187.2 mm, vias 0 -> 2
- net /MCU/ROW3: track 274.6 -> 93.1 mm
- net /MCU/COL8: track 0.00 -> 168.2 mm, vias 0 -> 2
- net /MCU/COL7: track 0.00 -> 148.6 mm, vias 0 -> 2
- net /MCU/COL6: track 0.00 -> 128.1 mm, vias 0 -> 2
- net /MCU/ROW4: track 0.00 -> 109.1 mm
- net /MCU/COL5: track 0.00 -> 109.0 mm, vias 0 -> 2
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Other:
- outline, holes or cut-outs redrawn
- copper layers 2 -> 4
- rule pad_to_mask_clearance: 0.051 -> 0.05
- rule solder_mask_min_width: 0.25 -> 0.05
- rule via_min_size: 0.4 -> 0.6

Commit message: More routing added planes and re-wired MCU a bit
Parts:
- moved C16 3.81 mm to (52.2, 51.7)
- moved C18 3.81 mm to (51.1, 51.7)
- moved C19 3.30 mm to (54.9, 49.1), turned to 0 degrees
- moved C6 2.84 mm to (64.8, 72.9)
- moved L2 2.22 mm to (52.7, 53.3), turned to 180 degrees
- moved C7 1.98 mm to (49.0, 66.0)
- moved C10 1.55 mm to (58.3, 58.2)
- moved C13 1.55 mm to (57.8, 59.7)
- moved C15 1.55 mm to (42.8, 54.1)
- moved C17 1.55 mm to (54.4, 50.8)
- moved L1 1.55 mm to (53.9, 54.5)
- moved R3 1.55 mm to (48.1, 57.1)
- moved U2 1.55 mm to (54.1, 57.9)
- moved C14 1.55 mm to (43.1, 59.9)
- moved L3 1.55 mm to (54.4, 52.8)
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Connections:
- J1 pad 10: Net-(J1-Pad10) -> /MCU/NRST
- J1 pad 6: Net-(J1-Pad6) -> /MCU/COL3
- SW32 pad 2: /MCU/COL3 -> /MCU/COL5
- SW36 pad 2: /MCU/COL4 -> /MCU/COL8
- SW40 pad 2: /MCU/COL5 -> /MCU/COL9
- SW44 pad 2: /MCU/COL6 -> /MCU/COL10
- SW48 pad 2: /MCU/COL7 -> /MCU/COL11
- SW52 pad 2: /MCU/COL8 -> /MCU/COL13
- SW65 pad 2: /MCU/COL12 -> /MCU/COL13
- U2 pad 21: (no net) -> GND
- U6 pad 9: (no net) -> GND
- U7 pad 7: (no net) -> GND
Routing:
- net /MCU/ROW0: track 30.1 -> 325.7 mm, vias 0 -> 2
- net /MCU/ROW3: track 93.1 -> 379.9 mm, vias 0 -> 2
- net /MCU/ROW4: track 109.1 -> 392.6 mm
- net /MCU/ROW1: track 51.0 -> 332.0 mm, vias 0 -> 2
- net /MCU/ROW2: track 71.1 -> 351.1 mm, vias 0 -> 2
- net GND: track 0.00 -> 187.4 mm, vias 4 -> 115
- net /MCU/COL11: track 228.4 -> 345.1 mm, vias 2 -> 6
- net /MCU/COL8: track 168.2 -> 282.7 mm, vias 2 -> 6
- net /MCU/COL10: track 207.0 -> 321.0 mm, vias 2 -> 6
- net /MCU/COL9: track 187.2 -> 298.9 mm, vias 2 -> 6
- net /MCU/COL1: track 29.5 -> 139.7 mm, vias 0 -> 5
- net /MCU/COL5: track 109.0 -> 214.6 mm, vias 2 -> 6
- net /MCU/COL2: track 48.0 -> 152.4 mm, vias 0 -> 6
- net /MCU/COL13: track 277.4 -> 380.9 mm, vias 2 -> 5
- net /MCU/COL0: track 11.0 -> 110.8 mm, vias 0 -> 5
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- added copper zone on In1.Cu, net +3V3
- added copper zone on In2.Cu, net GND
Other:
- net class Default: clearance 0.2 -> 0.152
- rule trace_clearance: 0.2 -> 0.152
- rule via_min_drill: 0.3 -> 0.2
- rule via_min_size: 0.6 -> 0.45

Commit message: Create gerbers picknplace and bom
Parts:
- added H1: MountingHole, MountingHole:MountingHole_4.3mm_M4, F.Cu at (76.5, 123.8)
- added H2: MountingHole, MountingHole:MountingHole_4.3mm_M4, F.Cu at (299.7, 84.2)
- added H3: MountingHole, MountingHole:MountingHole_4.3mm_M4, F.Cu at (141.9, 159.6)
- added H4: MountingHole, MountingHole:MountingHole_4.3mm_M4, F.Cu at (283.7, 134.2)
Routing:
- net /MCU/USB_D-: track 21.7 -> 22.5 mm

Commit message: Re-Generate Gerbers
Parts:
- D69, D73, D74, D75, D76, D77, D78, D79, D80, D81, D82, D83: footprint LED_SMD:LED_WS2812B_PLCC4_5.0x5.0mm_P3.2mm -> lib_fp:LED_WS2812B_PLCC4_5.0x5.0mm_P3.2mm
- R15, R6: value 1.1K -> 1.2K
- R8: value 820R -> 1K
- U7: footprint Package_DFN_QFN:DFN-6-1EP_3x3mm_P0.95mm_EP1.7x2.6mm -> lib_fp:DFN-6-1EP_3x3mm_P0.95mm_EP1.7x2.6mm
- turned U7 to 270 degrees
Other:
- board text added: "BUTTON"
- board text added: "OLED"
- board text added: "SMA CONNECTOR"
- board text added: "USB Connector"
